Commit message: prepare push

File: webots_ros2_universal_robot/resource/ur5e_with_gripper.urdf (robot description, URDF)
Before this commit: robot ur5e, 24 links, 23 joints
Links:
- link base_link_inertia: geometry collision mesh filename=package://resource/Universal_Robots_ROS2_Driver/ur_descript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; visual mesh filename=package://resource/Universal_Robots_ROS2_Driver/ur_descript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
- link finger_1_link_0: geometry collision mesh filename=package://resource/robotiq/robotiq_3f_gripper_visualization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; visual mesh filename=package://resource/robotiq/robotiq_3f_gripper_visualization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
- link finger_1_link_1: geometry collision mesh filename=package://resource/robotiq/robotiq_3f_gripper_visualization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; visual mesh filename=package://resource/robotiq/robotiq_3f_gripper_visualization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
- link finger_1_link_2: geometry collision mesh filename=package://resource/robotiq/robotiq_3f_gripper_visualization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; visual mesh filename=package://resource/robotiq/robotiq_3f_gripper_visualization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
- link finger_1_link_3: geometry collision mesh filename=package://resource/robotiq/robotiq_3f_gripper_visualization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; visual mesh filename=package://resource/robotiq/robotiq_3f_gripper_visualization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
- link finger_2_link_0: geometry collision mesh filename=package://resource/robotiq/robotiq_3f_gripper_visualization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; visual mesh filename=package://resource/robotiq/robotiq_3f_gripper_visualization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
- link finger_2_link_1: geometry collision mesh filename=package://resource/robotiq/robotiq_3f_gripper_visualization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; visual mesh filename=package://resource/robotiq/robotiq_3f_gripper_visualization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
- link finger_2_link_2: geometry collision mesh filename=package://resource/robotiq/robotiq_3f_gripper_visualization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; visual mesh filename=package://resource/robotiq/robotiq_3f_gripper_visualization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
- link finger_2_link_3: geometry collision mesh filename=package://resource/robotiq/robotiq_3f_gripper_visualization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; visual mesh filename=package://resource/robotiq/robotiq_3f_gripper_visualization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
- link finger_middle_link_0: geometry collision mesh filename=package://resource/robotiq/robotiq_3f_gripper_visualization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; visual mesh filename=package://resource/robotiq/robotiq_3f_gripper_visualization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
- link finger_middle_link_1: geometry collision mesh filename=package://resource/robotiq/robotiq_3f_gripper_visualization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; visual mesh filename=package://resource/robotiq/robotiq_3f_gripper_visualization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
- link finger_middle_link_2: geometry collision mesh filename=package://resource/robotiq/robotiq_3f_gripper_visualization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; visual mesh filename=package://resource/robotiq/robotiq_3f_gripper_visualization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
- link finger_middle_link_3: geometry collision mesh filename=package://resource/robotiq/robotiq_3f_gripper_visualization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; visual mesh filename=package://resource/robotiq/robotiq_3f_gripper_visualization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
- link forearm_link: geometry collision mesh filename=package://resource/Universal_Robots_ROS2_Driver/ur_descript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; visual mesh filename=package://resource/Universal_Robots_ROS2_Driver/ur_descript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
- link palm: geometry collision mesh filename=package://resource/robotiq/robotiq_3f_gripper_visualization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; visual mesh filename=package://resource/robotiq/robotiq_3f_gripper_visualization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
- link shoulder_link: geometry collision mesh filename=package://resource/Universal_Robots_ROS2_Driver/ur_descript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; visual mesh filename=package://resource/Universal_Robots_ROS2_Driver/ur_descript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
- link upper_arm_link: geometry collision mesh filename=package://resource/Universal_Robots_ROS2_Driver/ur_descript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; visual mesh filename=package://resource/Universal_Robots_ROS2_Driver/ur_descript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
- link wrist_1_link: geometry collision mesh filename=package://resource/Universal_Robots_ROS2_Driver/ur_descript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; visual mesh filename=package://resource/Universal_Robots_ROS2_Driver/ur_descript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
- link wrist_2_link: geometry collision mesh filename=package://resource/Universal_Robots_ROS2_Driver/ur_descript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; visual mesh filename=package://resource/Universal_Robots_ROS2_Driver/ur_descript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
- link wrist_3_link: geometry collision mesh filename=package://resource/Universal_Robots_ROS2_Driver/ur_descript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; visual mesh filename=package://resource/Universal_Robots_ROS2_Driver/ur_descript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
Joints:
- removed joint palm_tool0
- added joint tool0_palm: type fixed, parent tool0, child palm, origin xyz=0 0.045 0 rpy=1.5708 0 0

Commit message: enable conversion from robot_description

File: webots_ros2_universal_robot/resource/ur5e_with_gripper.urdf (robot description, URDF)
Before this commit: robot None, 24 links, 23 joints
Links:
- link base_link_inertia: geometry collision mesh filename=package://webots_ros2_universal_robot/resource/Universal_Ro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; visual mesh filename=package://webots_ros2_universal_robot/resource/Universal_Ro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
- link finger_1_link_0: geometry collision mesh filename=package://webots_ros2_universal_robot/resource/robotiq/robo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; visual mesh filename=package://webots_ros2_universal_robot/resource/robotiq/robo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
- link finger_1_link_1: geometry collision mesh filename=package://webots_ros2_universal_robot/resource/robotiq/robo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; visual mesh filename=package://webots_ros2_universal_robot/resource/robotiq/robo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
- link finger_1_link_2: geometry collision mesh filename=package://webots_ros2_universal_robot/resource/robotiq/robo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; visual mesh filename=package://webots_ros2_universal_robot/resource/robotiq/robo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
- link finger_1_link_3: geometry collision mesh filename=package://webots_ros2_universal_robot/resource/robotiq/robo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; visual mesh filename=package://webots_ros2_universal_robot/resource/robotiq/robo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
- link finger_2_link_0: geometry collision mesh filename=package://webots_ros2_universal_robot/resource/robotiq/robo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; visual mesh filename=package://webots_ros2_universal_robot/resource/robotiq/robo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
- link finger_2_link_1: geometry collision mesh filename=package://webots_ros2_universal_robot/resource/robotiq/robo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; visual mesh filename=package://webots_ros2_universal_robot/resource/robotiq/robo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
- link finger_2_link_2: geometry collision mesh filename=package://webots_ros2_universal_robot/resource/robotiq/robo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; visual mesh filename=package://webots_ros2_universal_robot/resource/robotiq/robo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
- link finger_2_link_3: geometry collision mesh filename=package://webots_ros2_universal_robot/resource/robotiq/robo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; visual mesh filename=package://webots_ros2_universal_robot/resource/robotiq/robo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
- link finger_middle_link_0: geometry collision mesh filename=package://webots_ros2_universal_robot/resource/robotiq/robo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; visual mesh filename=package://webots_ros2_universal_robot/resource/robotiq/robo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
- link finger_middle_link_1: geometry collision mesh filename=package://webots_ros2_universal_robot/resource/robotiq/robo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; visual mesh filename=package://webots_ros2_universal_robot/resource/robotiq/robo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
- link finger_middle_link_2: geometry collision mesh filename=package://webots_ros2_universal_robot/resource/robotiq/robo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; visual mesh filename=package://webots_ros2_universal_robot/resource/robotiq/robo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
- link finger_middle_link_3: geometry collision mesh filename=package://webots_ros2_universal_robot/resource/robotiq/robo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; visual mesh filename=package://webots_ros2_universal_robot/resource/robotiq/robo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
- link forearm_link: geometry collision mesh filename=package://webots_ros2_universal_robot/resource/Universal_Ro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; visual mesh filename=package://webots_ros2_universal_robot/resource/Universal_Ro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
- link palm: geometry collision mesh filename=package://webots_ros2_universal_robot/resource/robotiq/robo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; visual mesh filename=package://webots_ros2_universal_robot/resource/robotiq/robo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
- link shoulder_link: geometry collision mesh filename=package://webots_ros2_universal_robot/resource/Universal_Ro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; visual mesh filename=package://webots_ros2_universal_robot/resource/Universal_Ro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
- link upper_arm_link: geometry collision mesh filename=package://webots_ros2_universal_robot/resource/Universal_Ro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; visual mesh filename=package://webots_ros2_universal_robot/resource/Universal_Ro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
- link wrist_1_link: geometry collision mesh filename=package://webots_ros2_universal_robot/resource/Universal_Ro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; visual mesh filename=package://webots_ros2_universal_robot/resource/Universal_Ro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
- link wrist_2_link: geometry collision mesh filename=package://webots_ros2_universal_robot/resource/Universal_Ro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; visual mesh filename=package://webots_ros2_universal_robot/resource/Universal_Ro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
- link wrist_3_link: geometry collision mesh filename=package://webots_ros2_universal_robot/resource/Universal_Ro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; visual mesh filename=package://webots_ros2_universal_robot/resource/Universal_Ro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
