Commit message: moveit remove extra urdf

File: webots_ros2_universal_robot/resource/robotiq/robotiq_3f_gripper_visualization/cfg/robotiq-3f-gripper_articulated_macro.xacro (robot description, xacro)
@@ -60,5 +60,5 @@
     <parent link="${prefix}tool0"/>
     <child link="${prefix}palm"/>
-    <origin xyz="0 0.045 0" rpy="1.5708 0 0"/>
+    <origin xyz="0 0 0.045" rpy="1.5708 0 0"/>
 </joint>
 		<!-- end of joint list -->

File: webots_ros2_universal_robot/resource/ur5e_with_gripper.urdf (robot description, URDF)
Before this commit: robot None, 24 links, 23 joints
Joints:
- joint tool0_palm: origin xyz=0 0.045 0 rpy=1.5708 0 0 -> xyz=0 0 0.045 rpy=1.5708 0 0

File: webots_ros2_universal_robot/resource/ur5e_with_gripper.urdf.xacro (robot description, xacro)
@@ -1,4 +1,4 @@
 <?xml version="1.0"?>
-<robot xmlns:xacro="http://wiki.ros.org/xacro">
+<robot name="UR5e" xmlns:xacro="http://wiki.ros.org/xacro">
     <!-- Custom mix of ur5e robot and robotiq 3f gripper for Webots.
       Based on https://github.com/UniversalRobots/Universal_Robots_ROS2_Driver
