Commit message: fix tiago

File: webots_ros2_epuck/resource/epuck_webots.urdf (robot description, URDF)
Before this commit: robot Epuck Webots, 0 links, 0 joints
Links:
- added link base_link
- added link left_wheel_link
- added link right_wheel_link
Joints:
- added joint left wheel motor: type continuous, parent base_link, child left_wheel_link
- added joint right wheel motor: type continuous, parent base_link, child right_wheel_link

File: webots_ros2_tiago/resource/tiago_bringup_webots.urdf (robot description, URDF)
Before this commit: robot Tiago Webots, 0 links, 0 joints
Links:
- added link arm_1_link
- added link arm_2_link
- added link arm_3_link
- added link arm_4_link
- added link arm_5_link
- added link arm_6_link
- added link arm_7_link
- added link base_link
- added link gripper_left_finger_link
- added link gripper_right_finger_link
- added link head_1_link
- added link head_2_link
- added link torso_lift_link
- added link wheel_left_link
- added link wheel_right_link
Joints:
- added joint arm_1_joint: type continuous, parent torso_lift_link, child arm_1_link
- added joint arm_2_joint: type continuous, parent arm_1_link, child arm_2_link
- added joint arm_3_joint: type continuous, parent arm_2_link, child arm_3_link
- added joint arm_4_joint: type continuous, parent arm_3_link, child arm_4_link
- added joint arm_5_joint: type continuous, parent arm_4_link, child arm_5_link
- added joint arm_6_joint: type continuous, parent arm_5_link, child arm_6_link
- added joint arm_7_joint: type continuous, parent arm_6_link, child arm_7_link
- added joint gripper_left_finger_joint: type continuous, parent arm_7_link, child gripper_left_finger_link
- added joint gripper_right_finger_joint: type continuous, parent arm_7_link, child gripper_right_finger_link
- added joint head_1_joint: type continuous, parent base_link, child head_1_link
- added joint head_2_joint: type continuous, parent head_1_link, child head_2_link
- added joint torso_lift_joint: type continuous, parent base_link, child torso_lift_link
- added joint wheel_left_joint: type continuous, parent base_link, child wheel_left_link
- added joint wheel_right_joint: type continuous, parent base_link, child wheel_right_link

File: webots_ros2_tiago/resource/tiago_webots.urdf (robot description, URDF)
Before this commit: robot Tiago Webots, 0 links, 0 joints
Links:
- added link base_link
- added link wheel_left_link
- added link wheel_right_link
Joints:
- added joint wheel_left_joint: type continuous, parent base_link, child wheel_left_link
- added joint wheel_right_joint: type continuous, parent base_link, child wheel_right_link

Commit message: cleanup

File: webots_ros2_epuck/resource/epuck_webots.urdf (robot description, URDF)
Before this commit: robot Epuck Webots, 3 links, 2 joints
Links:
- removed link base_link
- removed link left_wheel_link
- removed link right_wheel_link
Joints:
- removed joint left wheel motor
- removed joint right wheel motor

File: webots_ros2_tiago/resource/tiago_bringup_webots.urdf (robot description, URDF)
Before this commit: robot Tiago Webots, 15 links, 14 joints
Links:
- removed link arm_1_link
- removed link arm_2_link
- removed link arm_3_link
- removed link arm_4_link
- removed link arm_5_link
- removed link arm_6_link
- removed link arm_7_link
- removed link base_link
- removed link gripper_left_finger_link
- removed link gripper_right_finger_link
- removed link head_1_link
- removed link head_2_link
- removed link torso_lift_link
- removed link wheel_left_link
- removed link wheel_right_link
Joints:
- removed joint arm_1_joint
- removed joint arm_2_joint
- removed joint arm_3_joint
- removed joint arm_4_joint
- removed joint arm_5_joint
- removed joint arm_6_joint
- removed joint arm_7_joint
- removed joint gripper_left_finger_joint
- removed joint gripper_right_finger_joint
- removed joint head_1_joint
- removed joint head_2_joint
- removed joint torso_lift_joint
- removed joint wheel_left_joint
- removed joint wheel_right_joint

File: webots_ros2_tiago/resource/tiago_webots.urdf (robot description, URDF)
Before this commit: robot Tiago Webots, 3 links, 2 joints
Links:
- removed link base_link
- removed link wheel_left_link
- removed link wheel_right_link
Joints:
- removed joint wheel_left_joint
- removed joint wheel_right_joint

File: webots_ros2_turtlebot/resource/turtlebot_webots.urdf (robot description, URDF)
Before this commit: robot TurtleBot3 Burger Webots, 3 links, 2 joints
Links:
- removed link base_link
- removed link left_wheel_link
- removed link right_wheel_link
Joints:
- removed joint left wheel motor
- removed joint right wheel motor
