Commit message: Removed redundant tags in urdf.

File: webots_ros2_tests/resource/connector_and_vacuum_gripper_test.urdf (robot description, URDF)
Before this commit: robot connector_and_vacuum_gripper_test_robot_webots, 3 links, 2 joints
Links:
- removed link base_link
- removed link connector_link
- removed link vacuum_gripper_link
Joints:
- removed joint connector_motor
- removed joint vacuum_gripper_motor
